File: schematics/kiCad/blinky-cube.kicad_pcb (KiCad board)
At the start: 2 copper layers, 86.6 x 49.7 mm, 14 parts, among them J1 Screw_Terminal_01x03, J2 Screw_Terminal_01x03, J3 Screw_Terminal_01x03, J4 Screw_Terminal_01x03, SW1 SW_Push, U1 Pico

Commit message: first commit
Parts:
- moved R3 20.3 mm to (132.4, 59.9)
- moved R4 14.5 mm to (122.0, 60.0)
- moved R5 10.0 mm to (122.2, 89.0), turned to -90 degrees
Connections:
- J1 pad 3: GND -> Net-(J1-Pin_3)
- J2 pad 3: GND -> Net-(J2-Pin_3)
- J3 pad 3: GND -> Net-(J3-Pin_3)
- R3 pad 2: Net-(J1-Pin_1) -> GND
- R4 pad 2: Net-(J3-Pin_1) -> GND
- R5 pad 2: Net-(J2-Pin_1) -> GND
- U1 pad 14: unconnected-(U1-GPIO10-Pad14) -> Net-(J1-Pin_1)
- U1 pad 15: Net-(J1-Pin_1) -> Net-(J1-Pin_2)
- U1 pad 16: Net-(J1-Pin_2) -> Net-(J1-Pin_3)
- U1 pad 17: unconnected-(U1-GPIO13-Pad17) -> Net-(J3-Pin_1)
- U1 pad 19: Net-(J3-Pin_1) -> Net-(J3-Pin_2)
- U1 pad 20: Net-(J3-Pin_2) -> Net-(J3-Pin_3)
- U1 pad 24: unconnected-(U1-GPIO18-Pad24) -> Net-(J2-Pin_3)
Routing:
- net Net-(J1-Pin_3): track 0.00 -> 35.9 mm
- net Net-(J2-Pin_3): track 0.00 -> 31.9 mm
- net Net-(J3-Pin_3): track 0.00 -> 23.8 mm
- net Net-(J3-Pin_1): track 25.5 -> 36.1 mm
- net Net-(J3-Pin_2): track 20.4 -> 29.8 mm
- net Net-(J1-Pin_2): track 31.0 -> 38.6 mm
- net Net-(J1-Pin_1): track 35.5 -> 40.0 mm
- net Net-(J2-Pin_2): track 20.3 -> 21.4 mm
- net GND: track 0.49 -> 0.00 mm, vias 7 -> 8
Other:
- board text added: "blinky-thermo-switch-p-cube v2.0"
- board text removed: "blinky-DS18B20-p-cube v2.0"
