File: schematics/kiCad/blinky-cube.kicad_sch (KiCad schematic)
At the start: 13 parts, among them J1 Screw_Terminal_01x03, J2 Screw_Terminal_01x03, J3 Screw_Terminal_01x03, J4 Screw_Terminal_01x03, SW1 SW_Push, U1 Pico

Commit message: first commit
Connections:
- net GND: now also R3.2, R4.2, R5.2; no longer J1.3 (Pin_3), J2.3 (Pin_3), J3.3 (Pin_3)
- net at U1.14 (GPIO10): now also J1.1 (Pin_1)
- net at J1.2 (Pin_2), R3.1: now also U1.15 (GPIO11); no longer U1.16 (GPIO12)
- net at U1.17 (GPIO13): now also J3.1 (Pin_1)
- net at J3.2 (Pin_2), R4.1: now also U1.19 (GPIO14); no longer U1.20 (GPIO15)
- net at J2.1 (Pin_1), U1.21 (GPIO16): no longer R5.2
- net at U1.24 (GPIO18): now also J2.3 (Pin_3)
- new net: J1.3 (Pin_3), U1.16 (GPIO12)
- new net: J3.3 (Pin_3), U1.20 (GPIO15)
- no-connect marks 22 -> 19
Other:
- note added: "blinky-thermo-switch-p-cube v2.0"
- note removed: "blinky-DS18B20-p-cube v2.0"
- moved on the sheet: J1, J2, J3, R3, R4, R5
